File: baraboard.kicad_pcb (KiCad board)
At the start: 2 copper layers, 26 parts, among them J1 OLED_128x64, U1 MCU_Seeed_XIAO_RP2040

Commit message: schema is done, pcb on the way
Parts:
- removed J1: OLED_128x64, ScottoKeebs_Components:OLED_128x64
- added D13: LED_WS2812B, ScottoKeebs_Components:LED_SK6812MINI, F.Cu at (141.9, 53.0)
- added D14: LED_WS2812B, ScottoKeebs_Components:LED_SK6812MINI, F.Cu at (160.9, 53.0)
- added D15: LED_WS2812B, ScottoKeebs_Components:LED_SK6812MINI, F.Cu at (180.0, 53.0)
- added D16: LED_WS2812B, ScottoKeebs_Components:LED_SK6812MINI, F.Cu at (141.9, 72.1)
- added D18: LED_WS2812B, ScottoKeebs_Components:LED_SK6812MINI, F.Cu at (160.9, 72.1)
- added D19: LED_WS2812B, ScottoKeebs_Components:LED_SK6812MINI, F.Cu at (180.0, 72.1)
- added D20: LED_WS2812B, ScottoKeebs_Components:LED_SK6812MINI, F.Cu at (141.9, 91.1)
- added D21: LED_WS2812B, ScottoKeebs_Components:LED_SK6812MINI, F.Cu at (160.9, 91.1)
- added D23: LED_WS2812B, ScottoKeebs_Components:LED_SK6812MINI, F.Cu at (180.0, 91.1)
- added D24: LED_WS2812B, ScottoKeebs_Components:LED_SK6812MINI, F.Cu at (122.8, 110.2)
- added D25: LED_WS2812B, ScottoKeebs_Components:LED_SK6812MINI, F.Cu at (151.4, 110.0)
- added D26: LED_WS2812B, ScottoKeebs_Components:LED_SK6812MINI, F.Cu at (180.0, 110.2)
- added SW2: RotaryEncoder_Switch, Rotary_Encoder:RotaryEncoder_Alps_EC11E-Switch_Vertical_H20mm, F.Cu at (114.0, 75.0)
Connections:
- U1 pad 11: unconnected-(U1-PA6_A10_D10_MOSI-Pad11) -> RGB
- U1 pad 13: Ground -> GND
- U1 pad 14: PInput -> +5V
- U1 pad 5: Net-(J1-SCL) -> EC11SW
- U1 pad 6: Net-(J1-SDA) -> EC11B
- U1 pad 7: unconnected-(U1-PB08_A6_D6_TX-Pad7) -> EC11A
Other:
- board outline added: 3.4 x 3 mm

Commit message: PCB done, case coming
Parts:
- moved D10 0.32 mm to (133.0, 107.6)
Connections:
- D16 pad 4: Net-(D15-DOUT) -> Net-(D16-DIN)
- D18 pad 2: Net-(D18-DOUT) -> Net-(D16-DIN)
- D18 pad 4: Net-(D16-DOUT) -> Net-(D18-DIN)
- D19 pad 2: Net-(D19-DOUT) -> Net-(D18-DIN)
- D19 pad 4: Net-(D18-DOUT) -> Net-(D15-DOUT)
- D20 pad 4: Net-(D19-DOUT) -> Net-(D16-DOUT)
- U1 pad 10: Col 0 -> Col 2
- U1 pad 5: EC11SW -> EC11A
- U1 pad 7: EC11A -> EC11SW
- U1 pad 8: Col 2 -> Col 0
Routing:
- net GND: track 0.00 -> 352.0 mm, vias 0 -> 10
- net +5V: track 0.00 -> 327.4 mm, vias 0 -> 13
- net RGB: track 0.00 -> 145.4 mm, vias 0 -> 2
- net Col 2: track 0.00 -> 131.6 mm
- net Col 1: track 0.00 -> 119.8 mm
- net Row 3: track 0.00 -> 118.6 mm
- net Col 0: track 0.00 -> 105.7 mm
- net Net-(D23-DOUT): track 0.00 -> 97.3 mm
- net Row 2: track 0.00 -> 97.1 mm
- net Row 1: track 0.00 -> 85.1 mm
- net Row 0: track 0.00 -> 65.9 mm
- net Net-(D15-DOUT): track 0.00 -> 34.6 mm
- net Net-(D16-DOUT): track 0.00 -> 34.0 mm, vias 0 -> 2
- net Net-(D18-DIN): track 0.00 -> 33.1 mm, vias 0 -> 2
- net Net-(D16-DIN): track 0.00 -> 32.7 mm, vias 0 -> 4
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- added copper zone on B.Cu, net (none)
- added copper zone on F.Cu, net (none)
Other:
- board size 3.4 x 3 mm -> 83.8 x 77.5 mm
- board text added: "Thanks to Newton!"
- board text added: "barab."
