File: baraboard.kicad_pcb (KiCad board)
At the start: 2 copper layers, 83.8 x 77.5 mm, 38 parts, among them SW2 RotaryEncoder_Switch, U1 MCU_Seeed_XIAO_RP2040

Commit message: PCB complete, case start
Parts:
- added G***: LOGO, LOGO, F.Cu at (113.9, 43.7)
- added REF**: Stabilizer_MX_2.00u, ScottoKeebs_Stabilizer:Stabilizer_MX_2.00u, F.Cu at (151.4, 104.1)
- S1, S10, S12, S2, S3, S4, S5, S6, S7, S8, S9: footprint ScottoKeebs_Hotswap:Hotswap_MX_Plated_1.00u -> ScottoKeebs_MX:MX_PCB_1.00u
- S11: footprint ScottoKeebs_Hotswap:Hotswap_MX_Plated_2.00u -> ScottoKeebs_MX:MX_PCB_2.00u
- SW2: footprint Rotary_Encoder:RotaryEncoder_Alps_EC11E-Switch_Vertical_H20mm -> ScottoKeebs_Scotto:Encoder_EC11_MX
- moved SW2 7.85 mm to (121.4, 77.7)
Routing:
- net Net-(D13-DOUT): track 18.9 -> 14.6 mm
- net Col 2: track 131.6 -> 135.8 mm
- net Col 0: track 105.7 -> 108.6 mm
- net Col 1: track 119.8 -> 122.5 mm
- net GND: track 352.0 -> 350.6 mm
