File: baraboard.kicad_sch (KiCad schematic)
At the start: 27 parts, among them J1 OLED_128x64, U1 MCU_Seeed_XIAO_RP2040

Commit message: schema is done, pcb on the way
Parts:
- removed D13: LED_SK6812MINI, ScottoKeebs_Components:LED_SK6812MINI, symbol ScottoKeebs:LED_SK6812MINI
- removed J1: OLED_128x64, ScottoKeebs_Components:OLED_128x64, symbol ScottoKeebs:OLED_128x64
- added D13, D14, D15, D16, D18, D19, D20, D21, D23, D24, D25, D26: LED_WS2812B, ScottoKeebs_Components:LED_SK6812MINI, symbol ScottoKeebs:LED_WS2812B
- added SW2: RotaryEncoder_Switch, Rotary_Encoder:RotaryEncoder_Alps_EC11E-Switch_Vertical_H20mm, symbol Device:RotaryEncoder_Switch
Connections:
- net RGB: now reaches U1.11 (PA6_A10_D10_MOSI)
- net RGB: now also D13.4 (DIN)
- net EC11A: now reaches U1.7 (PB08_A6_D6_TX)
- net EC11A: now also SW2.A
- net EC11SW: now reaches U1.5 (PA8_A4_D4_SDA)
- net EC11SW: now also SW2.S2
- net EC11B: now reaches U1.6 (PA9_A5_D5_SCL)
- net EC11B: now also SW2.B
- net Ground renamed GND
- net GND: now also D13.3 (VSS), D14.3 (VSS), D15.3 (VSS), D16.3 (VSS), D18.3 (VSS), D19.3 (VSS), D20.3 (VSS), D21.3 (VSS), D23.3 (VSS), D24.3 (VSS), D25.3 (VSS), D26.3 (VSS), SW2.C, SW2.S1
- net PInput renamed +5V
- net +5V: now also D13.1 (VDD), D14.1 (VDD), D15.1 (VDD), D16.1 (VDD), D18.1 (VDD), D19.1 (VDD), D20.1 (VDD), D21.1 (VDD), D23.1 (VDD), D24.1 (VDD), D25.1 (VDD), D26.1 (VDD)
- new net: D19.2 (DOUT), D20.4 (DIN)
- new net: D18.2 (DOUT), D19.4 (DIN)
- new net: D24.2 (DOUT), D25.4 (DIN)
- new net: D23.2 (DOUT), D24.4 (DIN)
- new net: D21.2 (DOUT), D23.4 (DIN)
- new net: D20.2 (DOUT), D21.4 (DIN)
- new net: D25.2 (DOUT), D26.4 (DIN)
- new net: D13.2 (DOUT), D14.4 (DIN)
- new net: D16.2 (DOUT), D18.4 (DIN)
- new net: D15.2 (DOUT), D16.4 (DIN)
- new net: D14.2 (DOUT), D15.4 (DIN)
- no-connect marks 0 -> 2
Other:
- moved on the sheet: D1, D10, D11, D12, D2, D3, D4, D5, D6, D7, D8, D9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

Commit message: PCB done, case coming
Connections:
- net Col 0: now also U1.8 (PB09_A7_D7_RX); no longer U1.10 (PA5_A9_D9_MISO)
- net Col 2: now also U1.10 (PA5_A9_D9_MISO); no longer U1.8 (PB09_A7_D7_RX)
- net EC11A: now also U1.5 (PA8_A4_D4_SDA); no longer U1.7 (PB08_A6_D6_TX)
- net EC11SW: now also U1.7 (PB08_A6_D6_TX); no longer U1.5 (PA8_A4_D4_SDA)
- net at D19.2 (DOUT): now also D18.4 (DIN); no longer D20.4 (DIN)
- net at D19.4 (DIN): now also D15.2 (DOUT); no longer D18.2 (DOUT)
- net at D16.2 (DOUT): now also D20.4 (DIN); no longer D18.4 (DIN)
- net at D16.4 (DIN): now also D18.2 (DOUT); no longer D15.2 (DOUT)
Other:
- moved on the sheet: D19
Changed lines of the file:
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@@
 	(wire
 		(pts
+			(xy 114.3 73.66) (xy 114.3 90.17)
+		)
+		(stroke
+			(width 0)
+			(type default)
+		)
+	)
+	(wire
+		(pts
 			(xy 132.08 170.18) (xy 132.08 162.56)
 		)
@@
 	(wire
 		(pts
-			(xy 114.3 73.66) (xy 114.3 90.17)
-		)
-		(stroke
-			(width 0)
-			(type default)
-		)
-	)
-	(wire
-		(pts
 			(xy 172.72 143.51) (xy 182.88 143.51)
 		)
@@
 	(global_label "Col 0"
 		(shape input)
-		(at 114.3 165.1 0)
+		(at 114.3 170.18 0)
 		(fields_autoplaced yes)
 		(effects
@@
 		)
 		(property "Intersheetrefs" "${INTERSHEET_REFS}"
-			(at 122.5465 165.1 0)
+			(at 122.5465 170.18 0)
 			(effects
 				(font
@@
 	(global_label "EC11A"
 		(shape input)
-		(at 73.66 170.18 180)
+		(at 73.66 165.1 180)
 		(fields_autoplaced yes)
 		(effects
@@
 		)
 		(property "Intersheetrefs" "${INTERSHEET_REFS}"
-			(at 64.7482 170.18 0)
+			(at 64.7482 165.1 0)
 			(effects
 				(font
@@
 	(global_label "EC11SW"
 		(shape input)
-		(at 73.66 165.1 180)
+		(at 73.66 170.18 180)
 		(fields_autoplaced yes)
 		(effects
@@
 		)
 		(property "Intersheetrefs" "${INTERSHEET_REFS}"
-			(at 63.1759 165.1 0)
+			(at 63.1759 170.18 0)
 			(effects
 				(font
@@
 	(global_label "Col 2"
 		(shape input)
-		(at 114.3 170.18 0)
+		(at 114.3 165.1 0)
 		(fields_autoplaced yes)
 		(effects
@@
 		)
 		(property "Intersheetrefs" "${INTERSHEET_REFS}"
-			(at 122.5465 170.18 0)
+			(at 122.5465 165.1 0)
 			(effects
 				(font
@@
 	(symbol
 		(lib_id "ScottoKeebs:LED_WS2812B")
-		(at 76.2 101.6 0)
+		(at 106.68 73.66 0)
 		(unit 1)
 		(exclude_from_sim no)
@@
 		(fields_autoplaced yes)
 		(property "Reference" "D19"
-			(at 88.9 95.2814 0)
+			(at 119.38 67.3414 0)
 			(effects
 				(font
@@
 		)
 		(property "Value" "LED_WS2812B"
-			(at 88.9 97.8214 0)
+			(at 119.38 69.8814 0)
 			(effects
 				(font
@@
 		)
 		(property "Footprint" "ScottoKeebs_Components:LED_SK6812MINI"
-			(at 77.47 109.22 0)
+			(at 107.95 81.28 0)
 			(effects
 				(font
@@
 		)
 		(property "Datasheet" "https://cdn-shop.adafruit.com/datasheets/WS2812B.pdf"
-			(at 78.74 111.125 0)
+			(at 109.22 83.185 0)
 			(effects
 				(font
@@
 		)
 		(property "Description" "RGB LED with integrated controller"
-			(at 76.2 101.6 0)
+			(at 106.68 73.66 0)
 			(effects
 				(font
@@
 	(symbol
 		(lib_id "power:GND")
-		(at 106.68 81.28 0)
+		(at 76.2 109.22 0)
 		(unit 1)
 		(exclude_from_sim no)
@@
 		(fields_autoplaced yes)
 		(property "Reference" "#PWR05"
-			(at 106.68 87.63 0)
+			(at 76.2 115.57 0)
 			(effects
 				(font
@@
 		)
 		(property "Value" "GND"
-			(at 106.68 86.36 0)
+			(at 76.2 114.3 0)
 			(effects
 				(font
@@
 		)
 		(property "Footprint" ""
-			(at 106.68 81.28 0)
+			(at 76.2 109.22 0)
 			(effects
 				(font
@@
 		)
 		(property "Datasheet" ""
-			(at 106.68 81.28 0)
+			(at 76.2 109.22 0)
 			(effects
 				(font
@@
 		)
 		(property "Description" "Power symbol creates a global label with name \"GND\" , ground"
-			(at 106.68 81.28 0)
+			(at 76.2 109.22 0)
 			(effects
 				(font
@@
 	(symbol
 		(lib_id "power:+5V")
-		(at 76.2 93.98 0)
+		(at 106.68 66.04 0)
 		(unit 1)
 		(exclude_from_sim no)
@@
 		(fields_autoplaced yes)
 		(property "Reference" "#PWR013"
-			(at 76.2 97.79 0)
+			(at 106.68 69.85 0)
 			(effects
 				(font
@@
 		)
 		(property "Value" "+5V"
-			(at 76.2 88.9 0)
+			(at 106.68 60.96 0)
 			(effects
 				(font
@@
 		)
 		(property "Footprint" ""
-			(at 76.2 93.98 0)
+			(at 106.68 66.04 0)
 			(effects
 				(font
@@
 		)
 		(property "Datasheet" ""
-			(at 76.2 93.98 0)
+			(at 106.68 66.04 0)
 			(effects
 				(font
@@
 		)
 		(property "Description" "Power symbol creates a global label with name \"+5V\""
-			(at 76.2 93.98 0)
+			(at 106.68 66.04 0)
 			(effects
 				(font
@@
 	(symbol
 		(lib_id "power:GND")
-		(at 76.2 109.22 0)
+		(at 106.68 81.28 0)
 		(unit 1)
 		(exclude_from_sim no)
@@
 		(fields_autoplaced yes)
 		(property "Reference" "#PWR014"
-			(at 76.2 115.57 0)
+			(at 106.68 87.63 0)
 			(effects
 				(font
@@
 		)
 		(property "Value" "GND"
-			(at 76.2 114.3 0)
+			(at 106.68 86.36 0)
 			(effects
 				(font
@@
 		)
 		(property "Footprint" ""
-			(at 76.2 109.22 0)
+			(at 106.68 81.28 0)
 			(effects
 				(font
@@
 		)
 		(property "Datasheet" ""
-			(at 76.2 109.22 0)
+			(at 106.68 81.28 0)
 			(effects
 				(font
@@
 		)
 		(property "Description" "Power symbol creates a global label with name \"GND\" , ground"
-			(at 76.2 109.22 0)
+			(at 106.68 81.28 0)
 			(effects
 				(font
@@
 	(symbol
 		(lib_id "ScottoKeebs:LED_WS2812B")
-		(at 106.68 73.66 0)
+		(at 76.2 101.6 0)
 		(unit 1)
 		(exclude_from_sim no)
@@
 		(fields_autoplaced yes)
 		(property "Reference" "D16"
-			(at 119.38 67.3414 0)
+			(at 88.9 95.2814 0)
 			(effects
 				(font
@@
 		)
 		(property "Value" "LED_WS2812B"
-			(at 119.38 69.8814 0)
+			(at 88.9 97.8214 0)
 			(effects
 				(font
@@
 		)
 		(property "Footprint" "ScottoKeebs_Components:LED_SK6812MINI"
-			(at 107.95 81.28 0)
+			(at 77.47 109.22 0)
 			(effects
 				(font
@@
 		)
 		(property "Datasheet" "https://cdn-shop.adafruit.com/datasheets/WS2812B.pdf"
-			(at 109.22 83.185 0)
+			(at 78.74 111.125 0)
 			(effects
 				(font
@@
 		)
 		(property "Description" "RGB LED with integrated controller"
-			(at 106.68 73.66 0)
+			(at 76.2 101.6 0)
 			(effects
 				(font
@@
 		(on_board yes)
 		(dnp no)
-		(fields_autoplaced yes)
 		(property "Reference" "D15"
-			(at 104.14 67.3414 0)
+			(at 73.66 95.2814 0)
 			(effects
 				(font
@@
 		)
 		(property "Value" "LED_WS2812B"
-			(at 104.14 69.8814 0)
+			(at 104.14 57.1814 0)
 			(effects
 				(font
@@
 		(on_board yes)
 		(dnp no)
-		(fields_autoplaced yes)
 		(property "Reference" "#PWR07"
 			(at 76.2 69.85 0)
@@
 		)
 		(property "Value" "+5V"
-			(at 76.2 60.96 0)
+			(at 105.41 83.82 0)
 			(effects
 				(font
@@
 		(on_board yes)
 		(dnp no)
-		(fields_autoplaced yes)
 		(property "Reference" "D18"
-			(at 73.66 95.2814 0)
+			(at 104.14 67.3414 0)
 			(effects
 				(font
@@
 		)
 		(property "Value" "LED_WS2812B"
-			(at 73.66 97.8214 0)
+			(at 104.14 69.8814 0)
 			(effects
 				(font
@@
 	(symbol
 		(lib_id "power:+5V")
-		(at 106.68 66.04 0)
+		(at 76.2 93.98 0)
 		(unit 1)
 		(exclude_from_sim no)
@@
 		(fields_autoplaced yes)
 		(property "Reference" "#PWR09"
-			(at 106.68 69.85 0)
+			(at 76.2 97.79 0)
 			(effects
 				(font
@@
 		)
 		(property "Value" "+5V"
-			(at 106.68 60.96 0)
+			(at 76.2 88.9 0)
 			(effects
 				(font
@@
 		)
 		(property "Footprint" ""
-			(at 106.68 66.04 0)
+			(at 76.2 93.98 0)
 			(effects
 				(font
@@
 		)
 		(property "Datasheet" ""
-			(at 106.68 66.04 0)
+			(at 76.2 93.98 0)
 			(effects
 				(font
@@
 		)
 		(property "Description" "Power symbol creates a global label with name \"+5V\""
-			(at 106.68 66.04 0)
+			(at 76.2 93.98 0)
 			(effects
 				(font

Commit message: PCB complete, case start
Parts:
- S1, S10, S12, S2, S3, S4, S5, S6, S7, S8, S9: footprint ScottoKeebs_Hotswap:Hotswap_MX_Plated_1.00u -> ScottoKeebs_MX:MX_PCB_1.00u
- S11: footprint ScottoKeebs_Hotswap:Hotswap_MX_Plated_2.00u -> ScottoKeebs_MX:MX_PCB_2.00u
- SW2: footprint Rotary_Encoder:RotaryEncoder_Alps_EC11E-Switch_Vertical_H20mm -> ScottoKeebs_Scotto:Encoder_EC11_MX
Changed lines of the file:
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@@
 			)
 		)
-		(property "Footprint" "ScottoKeebs_Hotswap:Hotswap_MX_Plated_1.00u"
+		(property "Footprint" "ScottoKeebs_MX:MX_PCB_1.00u"
 			(at 160.02 113.03 0)
 			(effects
@@
 			)
 		)
-		(property "Footprint" "ScottoKeebs_Hotswap:Hotswap_MX_Plated_1.00u"
+		(property "Footprint" "ScottoKeebs_MX:MX_PCB_1.00u"
 			(at 160.02 133.35 0)
 			(effects
@@
 			)
 		)
-		(property "Footprint" "ScottoKeebs_Hotswap:Hotswap_MX_Plated_1.00u"
+		(property "Footprint" "ScottoKeebs_MX:MX_PCB_1.00u"
 			(at 160.02 74.93 0)
 			(effects
@@
 			)
 		)
-		(property "Footprint" "Rotary_Encoder:RotaryEncoder_Alps_EC11E-Switch_Vertical_H20mm"
+		(property "Footprint" "ScottoKeebs_Scotto:Encoder_EC11_MX"
 			(at 148.59 164.084 0)
 			(effects
@@
 			)
 		)
-		(property "Footprint" "ScottoKeebs_Hotswap:Hotswap_MX_Plated_1.00u"
+		(property "Footprint" "ScottoKeebs_MX:MX_PCB_1.00u"
 			(at 170.18 113.03 0)
 			(effects
@@
 			)
 		)
-		(property "Footprint" "ScottoKeebs_Hotswap:Hotswap_MX_Plated_1.00u"
+		(property "Footprint" "ScottoKeebs_MX:MX_PCB_1.00u"
 			(at 180.34 93.98 0)
 			(effects
@@
 			)
 		)
-		(property "Footprint" "ScottoKeebs_Hotswap:Hotswap_MX_Plated_1.00u"
+		(property "Footprint" "ScottoKeebs_MX:MX_PCB_1.00u"
 			(at 160.02 93.98 0)
 			(effects
@@
 			)
 		)
-		(property "Footprint" "ScottoKeebs_Hotswap:Hotswap_MX_Plated_1.00u"
+		(property "Footprint" "ScottoKeebs_MX:MX_PCB_1.00u"
 			(at 170.18 74.93 0)
 			(effects
@@
 			)
 		)
-		(property "Footprint" "ScottoKeebs_Hotswap:Hotswap_MX_Plated_2.00u"
+		(property "Footprint" "ScottoKeebs_MX:MX_PCB_2.00u"
 			(at 170.18 133.35 0)
 			(effects
@@
 			)
 		)
-		(property "Footprint" "ScottoKeebs_Hotswap:Hotswap_MX_Plated_1.00u"
+		(property "Footprint" "ScottoKeebs_MX:MX_PCB_1.00u"
 			(at 180.34 133.35 0)
 			(effects
@@
 			)
 		)
-		(property "Footprint" "ScottoKeebs_Hotswap:Hotswap_MX_Plated_1.00u"
+		(property "Footprint" "ScottoKeebs_MX:MX_PCB_1.00u"
 			(at 180.34 113.03 0)
 			(effects
@@
 			)
 		)
-		(property "Footprint" "ScottoKeebs_Hotswap:Hotswap_MX_Plated_1.00u"
+		(property "Footprint" "ScottoKeebs_MX:MX_PCB_1.00u"
 			(at 170.18 93.98 0)
 			(effects
@@
 			)
 		)
-		(property "Footprint" "ScottoKeebs_Hotswap:Hotswap_MX_Plated_1.00u"
+		(property "Footprint" "ScottoKeebs_MX:MX_PCB_1.00u"
 			(at 180.34 74.93 0)
 			(effects
